Commit message: added mass to the tip link of the fingers in the pro version urdfs

File: python/rrc_simulation/robot_properties_fingers/urdf/pro/fingerpro.urdf (robot description, URDF)
Before this commit: robot fingerpro, 6 links, 5 joints
Links:
- link finger_tip_link: mass 0 -> 0.02

File: python/rrc_simulation/robot_properties_fingers/urdf/pro/trifingerpro.urdf (robot description, URDF)
Before this commit: robot trifingerpro, 17 links, 16 joints
Links:
- link finger_tip_link_0: mass 0 -> 0.02
- link finger_tip_link_120: mass 0 -> 0.02
- link finger_tip_link_240: mass 0 -> 0.02

File: python/rrc_simulation/robot_properties_fingers/urdf/pro/trifingerpro_with_stage.urdf (robot description, URDF)
Before this commit: robot trifingerpro_with_stage, 19 links, 18 joints
Links:
- link finger_tip_link_0: mass 0 -> 0.02
- link finger_tip_link_120: mass 0 -> 0.02
- link finger_tip_link_240: mass 0 -> 0.02
